Commit message: ~4.5 orientation error fixed between ft300 and s_model gripper

File: robotiq_s_gripper/robotiq_s_model_control/urdf/s_model_open.urdf.xacro (robot description, xacro)
@@ -4,6 +4,8 @@
         <!-- mount the Gripper to the robot -->
         <joint name="${prefix}_s_model_adapter" type="fixed" >
-            <origin xyz="0.0 0.0 0.015" rpy="0.0 0.0 0.0"/>
-	    <parent link="${parent}" />
+            <!-- <origin xyz="0.0 0.0 0.015" rpy="0.0 0.0 3.14159"/> -->
+            <!-- This new origin corrects ~4.5deg (0.0785rad) error in the gripper pose wrt ft300 -->
+            <origin xyz="0.0 0.0 0.015" rpy="0.0 0.0 3.22013"/>
+            <parent link="${parent}" />
             <child link="${prefix}s_model_adapter_link" />
         </joint>
