Commit message: urdf for arm realsense d415 added to config

File: husky_description/urdf/accessories/husky_ur_accessories.urdf.xacro (robot description, xacro)
@@ -4,4 +4,6 @@
   <xacro:include filename="$(find robotiq_s_model_control)/urdf/s_model_open.urdf.xacro" />
   <xacro:include filename="$(find robotiq_c_model_viz)/urdf/c_model_open.urdf.xacro" />
+  <!-- RealSense D41X Camera -->
+  <xacro:include filename="$(find realsense_ros_camera)/urdf/_r410.urdf.xacro"/>
   <!-- CHANGE BELOW VALUES DURING INTEGRATION -->
   <!-- MUST CHANGE TO UR5, UR3 or UR10 depending on needs -->
@@ -11,5 +13,5 @@
   <xacro:arg name="ur10_enabled" default="false"/>
   <xacro:property name="ur_origin">
-   <origin xyz="0.28 0 0.0065" rpy="0.0 0.0 -1.57" />
+    <origin xyz="0.28 0 0.0065" rpy="0.0 0.0 -1.5708" />
   </xacro:property>
   <xacro:arg name="ft_300_enabled" default="true"/>
@@ -26,52 +28,78 @@
   </xacro:property>
   <!-- CHANGE ABOVE VALUES DURING INTEGRATION -->
-    <xacro:if value="$(arg ft_300_enabled)">
-      <!-- Spawn FT Sensor -->
-      <xacro:robotiq_fts300 prefix="$(arg ft_300_prefix)" parent="$(arg ft_300_parent)" />
-    </xacro:if>
-    <xacro:if value="$(arg s_model_enabled)">
-      <!-- Spawn S model Gripper -->
-      <xacro:s_model_open prefix="$(arg s_model_prefix)" parent="$(arg s_model_parent)"/>
-    </xacro:if>
-    <xacro:if value="$(arg c_model_enabled)">
-      <!-- Spawn S model Gripper -->
-      <xacro:c_model_open prefix="$(arg c_model_prefix)" parent="$(arg c_model_parent)"/>
-    </xacro:if>
-    <xacro:if value="$(arg ur3_enabled)">
-      <!-- Spawn arm -->
-      <xacro:ur3_robot prefix="ur_arm_" joint_limited="true"/>
-    </xacro:if>
-    <xacro:if value="$(arg ur5_enabled)">
-      <!-- Spawn arm -->
-      <xacro:ur5_robot prefix="ur_arm_" joint_limited="true"/>
-    </xacro:if>
-    <xacro:if value="$(arg ur10_enabled)">
-      <!-- Spawn arm -->
-      <xacro:ur10_robot prefix="ur_arm_" joint_limited="true"/>
-    </xacro:if>
-      <!-- Join arm -->
-      <joint name="ur_arm_base" type="fixed">
-        <parent link="top_plate_link" />
-        <child link="ur_arm_base_link" />
-        <xacro:insert_block name="ur_origin" />
-      </joint>
-    <!-- Spawn the sensor arch link -->
-      <link name="sensor_arch_mount_link">
-             <visual>
-                 <geometry>
-                     <mesh filename="package://husky_description/meshes/integration_arch.dae" />
-                 </geometry>
-             </visual>
-             <collision>
-                 <geometry>
-                     <mesh filename="package://husky_description/meshes/integration_arch.dae" />
-                 </geometry>
-             </collision>
-    </link>
-    <!-- Attach the sensor arch to the top plate -->
-    <joint name="sensor_arch_mount" type="fixed">
-             <parent link="top_plate_link"/>
-             <child link="sensor_arch_mount_link"/>
-             <xacro:insert_block name="arch_origin" />
-    </joint>
+  <xacro:if value="$(arg ft_300_enabled)">
+    <!-- Spawn FT Sensor -->
+    <xacro:robotiq_fts300 prefix="$(arg ft_300_prefix)" parent="$(arg ft_300_parent)" />
+  </xacro:if>
+  <xacro:if value="$(arg s_model_enabled)">
+    <!-- Spawn S model Gripper -->
+    <xacro:s_model_open prefix="$(arg s_model_prefix)" parent="$(arg s_model_parent)"/>
+  </xacro:if>
+  <xacro:if value="$(arg c_model_enabled)">
+    <!-- Spawn C model Gripper -->
+    <xacro:c_model_open prefix="$(arg c_model_prefix)" parent="$(arg c_model_parent)"/>
+  </xacro:if>
+  <xacro:if value="$(arg ur3_enabled)">
+    <!-- Spawn arm -->
+    <xacro:ur3_robot prefix="ur_arm_" joint_limited="true"/>
+  </xacro:if>
+  <xacro:if value="$(arg ur5_enabled)">
+    <!-- Spawn arm -->
+    <xacro:ur5_robot prefix="ur_arm_" joint_limited="true"/>
+  </xacro:if>
+  <xacro:if value="$(arg ur10_enabled)">
+    <!-- Spawn arm -->
+    <xacro:ur10_robot prefix="ur_arm_" joint_limited="true"/>
+  </xacro:if>
+  <!-- Join arm -->
+  <joint name="ur_arm_base" type="fixed">
+    <parent link="top_plate_link" />
+    <child link="ur_arm_base_link" />
+    <xacro:insert_block name="ur_origin" />
+  </joint>
+  <!-- Spawn the sensor arch link -->
+  <link name="sensor_arch_mount_link">
+    <visual>
+      <geometry>
+        <mesh filename="package://husky_description/meshes/integration_arch.dae" />
+      </geometry>
+    </visual>
+    <collision>
+      <geometry>
+        <mesh filename="package://husky_description/meshes/integration_arch.dae" />
+      </geometry>
+    </collision>
+  </link>
+  <!-- Attach the sensor arch to the top plate -->
+  <joint name="sensor_arch_mount" type="fixed">
+    <parent link="top_plate_link"/>
+    <child link="sensor_arch_mount_link"/>
+    <xacro:insert_block name="arch_origin" />
+  </joint>
+  <!-- RealSense D41X Camera -->
+  <!-- <link name="arm_camera_link"/>
+  <joint name="arm_camera_joint" type="fixed">
+    <origin xyz="0.0 0.0 0.075" rpy="-1.5708 0 0"/>
+    <parent link="UR_1_s_model_link" />
+    <child link="arm_camera_link" />
+  </joint> -->
+  <!-- Spawn D415 camera -->
+  <sensor_r410 parent="UR_1_s_model_link" prefix="arm_">
+    <origin xyz="0 0 0.07" rpy="0 0 1.5708"/>
+  </sensor_r410>
+  <!-- Define optical_frame wrt the camera_link -->
+  <link name="/camera_arm/camera_color_optical_frame"/>
+  <joint name="/camera_arm/camera_color_optical_frame_joint" type="fixed">
+    <!-- <origin xyz="-0.05 0.0 0.02" rpy="0.0 0.0 0.06"/> -->
+    <origin xyz="0.0 0.0 0.075" rpy="-1.5708 0 0"/>
+    <parent link="UR_1_s_model_link" />
+    <child link="/camera_arm/camera_color_optical_frame" />
+  </joint>
+  <!-- Finger tip - Model S Gripper -->
+  <link name="hand_finger_tip_link"/>
+  <joint name="hand_finger_tip_joint" type="fixed">
+    <origin xyz="0.27 0 0" rpy="2.35619 0 0"/>
+    <parent link="ur_arm_ee_link" />
+    <child link="hand_finger_tip_link" />
+  </joint>
 </robot>

Commit message: added 3 move groups for planning wrt hand palm, hand center, and finger tip of model 2 gripper

File: husky_description/urdf/accessories/husky_ur_accessories.urdf.xacro (robot description, xacro)
@@ -78,11 +78,4 @@
   </joint>
   <!-- RealSense D41X Camera -->
-  <!-- <link name="arm_camera_link"/>
-  <joint name="arm_camera_joint" type="fixed">
-    <origin xyz="0.0 0.0 0.075" rpy="-1.5708 0 0"/>
-    <parent link="UR_1_s_model_link" />
-    <child link="arm_camera_link" />
-  </joint> -->
-  <!-- Spawn D415 camera -->
   <sensor_r410 parent="UR_1_s_model_link" prefix="arm_">
     <origin xyz="0 0 0.07" rpy="0 0 1.5708"/>
@@ -96,9 +89,23 @@
     <child link="/camera_arm/camera_color_optical_frame" />
   </joint>
+  <!-- Palm - Model S Gripper -->
+  <link name="hand_palm_link"/>
+  <joint name="hand_palm_joint" type="fixed">
+    <origin xyz="0.16 0 0" rpy="2.35619 0 0"/>
+    <parent link="ur_arm_ee_link" />
+    <child link="hand_palm_link" />
+  </joint>
+  <!-- Hand center - Model S Gripper -->
+  <link name="hand_center_link"/>
+  <joint name="hand_center_joint" type="fixed">
+    <origin xyz="0.055 0 0" rpy="0 0 0"/>
+    <parent link="hand_palm_link" />
+    <child link="hand_center_link" />
+  </joint>
   <!-- Finger tip - Model S Gripper -->
   <link name="hand_finger_tip_link"/>
   <joint name="hand_finger_tip_joint" type="fixed">
-    <origin xyz="0.27 0 0" rpy="2.35619 0 0"/>
-    <parent link="ur_arm_ee_link" />
+    <origin xyz="0.055 0 0" rpy="0 0 0"/>
+    <parent link="hand_center_link" />
     <child link="hand_finger_tip_link" />
   </joint>

Commit message: updated arm camera pose in urdf

File: husky_description/urdf/accessories/husky_ur_accessories.urdf.xacro (robot description, xacro)
@@ -84,6 +84,10 @@
   <link name="/camera_arm/camera_color_optical_frame"/>
   <joint name="/camera_arm/camera_color_optical_frame_joint" type="fixed">
-    <!-- <origin xyz="-0.05 0.0 0.02" rpy="0.0 0.0 0.06"/> -->
-    <origin xyz="0.0 0.0 0.075" rpy="-1.5708 0 0"/>
+    <!-- TODO: Old mount (manually calibrated): -->
+    <!-- <origin xyz="-0.05 0.0 0.08" rpy="-1.5708 0 0"/> -->
+    <!-- TODO: New mount (manually calibrated): -->
+    <!-- <origin xyz="-0.05 0.02 0.09" rpy="-1.561 0 -0.024"/> -->
+    <!-- TODO: New mount (automatically calibrated using visual triangulation): -->
+    <origin xyz="-0.0418 0.0156 0.0721" rpy="-1.5385 -0.0670 -0.0043"/>
     <parent link="UR_1_s_model_link" />
     <child link="/camera_arm/camera_color_optical_frame" />

Commit message: Added an independentController script to control individual fingers; added `UR_1_s_grip_point` link to the urdf.

File: husky_description/urdf/accessories/husky_ur_accessories.urdf.xacro (robot description, xacro)
@@ -114,3 +114,11 @@
     <child link="hand_finger_tip_link" />
   </joint>
+<!-- mount the grip point link under the UR_1_fts_toolside link. This is used for the compliance controller. Added by Vincent at Mar 24 2025 -->
+  <link name="UR_1_s_grip_point" />
+  <joint name="UR_1_s_grip_point_joint" type="fixed">
+    <parent link="UR_1_fts_toolside"/>
+    <child link="UR_1_s_grip_point"/>
+    <!-- z axis towards the gripper; rotate -45 degree to get axis-aligned pose -->
+    <origin xyz="0 0 0.20" rpy="0 0 -0.7854"/>
+  </joint>
 </robot>
